Commit message: Robot can turn to left and right.  + Adding left/right middle wheel, in order to make turnaroud possible  + Using diffdrive_multiwheel plugin from Hector to realize 6 wheel drive

File: ar2a_description/urdf/ar2a.xacro (robot description, xacro)
@@ -6,7 +6,5 @@
   <xacro:property name="chassisLength" value="0.45"/>
   <xacro:property name="chassisWidth" value="0.25"/>
-  <xacro:property name="chassisMass" value="60"/>
-  <xacro:property name="casterRadius" value="0.05"/>
-  <xacro:property name="casterMass" value="5"/>
+  <xacro:property name="chassisMass" value="6"/>
   <xacro:property name="wheelWidth" value="0.05"/>
   <xacro:property name="wheelRadius" value="0.05"/>
@@ -21,4 +19,5 @@
   <xacro:include filename="$(find ar2a_description)/urdf/materials.xacro" />
   <xacro:include filename="$(find ar2a_description)/urdf/macros.xacro" />
+  <xacro:include filename="$(find ar2a_description)/urdf/kinect.xacro" />
   <link name="footprint" />
   <joint name="base_joint" type="fixed">
@@ -46,91 +45,10 @@
     </inertial>
   </link>
-  <wheel lr="left_front" fb="1" tY="1"/>
-  <wheel lr="right_front" fb="1" tY="-1"/>
-  <wheel lr="left_back" fb="-1" tY="1"/>
-  <wheel lr="right_back" fb="-1" tY="-1"/>
-  <!-- Kinect Camera -->
-  <joint name="kinect_camera_joint" type="fixed">
-    <axis xyz="0 1 0" />
-    <origin xyz="${cameraPosX} ${cameraPosY} ${cameraPosZ}" rpy="0 0 0"/>
-    <parent link="chassis" />
-    <child link="camera_link" />
-  </joint>
-  <link name="camera_link">
-    <inertial>
-      <mass value="0.01" />
-      <origin xyz="${cameraPosX} ${cameraPosY} ${cameraPosZ}" />
-      <inertia ixx="0.001" ixy="0.0" ixz="0.0"
-       iyy="0.001" iyz="0.0"
-       izz="0.001" />
-    </inertial>
-    <visual>
-      <origin xyz="${cameraPosX} ${cameraPosY} ${cameraPosZ}" rpy="0 0 0" />
-      <geometry>
-        <mesh filename="package://ar2a_description/meshes/kinect.dae"/>
-      </geometry>
-    </visual>
-    <collision>
-      <origin xyz="${cameraPosX} ${cameraPosY} ${cameraPosZ}" rpy="0 0 0" />
-      <geometry>
-        <mesh filename="package://ar2a_description/meshes/kinect.dae"/>
-      </geometry>
-    </collision>
-  </link>
-  <joint name="camera_depth_joint" type="fixed">
-    <origin xyz="0 0.018 0" rpy="0 0 0" />
-    <parent link="camera_link" />
-    <child link="camera_depth_frame" />
-  </joint>
-  <link name="camera_depth_frame">
-    <inertial>
-      <mass value="0.01" />
-      <origin xyz="0 0 0" />
-      <inertia ixx="0.001" ixy="0.0" ixz="0.0"
-       iyy="0.001" iyz="0.0"
-       izz="0.001" />
-    </inertial>
-  </link>
-  <joint name="camera_depth_optical_joint" type="fixed">
-    <origin xyz="0 0 0" rpy="${-PI/2} 0 ${-PI/2}" />
-    <parent link="camera_depth_frame" />
-    <child link="camera_depth_optical_frame" />
-  </joint>
-  <link name="camera_depth_optical_frame">
-    <inertial>
-      <mass value="0.001" />
-      <origin xyz="0 0 0" />
-      <inertia ixx="0.0001" ixy="0.0" ixz="0.0"
-       iyy="0.0001" iyz="0.0"
-       izz="0.0001" />
-    </inertial>
-  </link>
-  <joint name="camera_rgb_joint" type="fixed">
-    <origin xyz="0 -0.005 0" rpy="0 0 0" />
-    <parent link="camera_link" />
-    <child link="camera_rgb_frame" />
-  </joint>
-  <link name="camera_rgb_frame">
-    <inertial>
-      <mass value="0.001" />
-      <origin xyz="0 0 0" />
-      <inertia ixx="0.0001" ixy="0.0" ixz="0.0"
-       iyy="0.0001" iyz="0.0"
-       izz="0.0001" />
-    </inertial>
-  </link>
-  <joint name="camera_rgb_optical_joint" type="fixed">
-    <origin xyz="0 0 0" rpy="${-PI/2} 0 ${-PI/2}" />
-    <parent link="camera_rgb_frame" />
-    <child link="camera_rgb_optical_frame" />
-  </joint>
-  <link name="camera_rgb_optical_frame">
-    <inertial>
-      <mass value="0.001" />
-      <origin xyz="0 0 0" />
-      <inertia ixx="0.0001" ixy="0.0" ixz="0.0"
-       iyy="0.0001" iyz="0.0"
-       izz="0.0001" />
-    </inertial>
-  </link>
+  <wheel lr="left_front" x_pos="${wheelPos}" y_pos="${wheelWidth/2+chassisWidth/2}"/>
+  <wheel lr="left_middle" x_pos="0.0" y_pos="${wheelWidth/2+chassisWidth/2}"/>
+  <wheel lr="left_back" x_pos="${-wheelPos}" y_pos="${wheelWidth/2+chassisWidth/2}"/>
+  <wheel lr="right_front" x_pos="${wheelPos}" y_pos="${-wheelWidth/2-chassisWidth/2}"/>
+  <wheel lr="right_middle" x_pos="0.0" y_pos="${-wheelWidth/2-chassisWidth/2}"/>
+  <wheel lr="right_back" x_pos="${-wheelPos}" y_pos="${-wheelWidth/2-chassisWidth/2}"/>
+  <kinect_camera/>
 </robot>

File: ar2a_description/urdf/macros.xacro (robot description, xacro)
@@ -22,9 +22,9 @@
     />
   </macro>
-  <!-- params = left/right front/back translation Y-Axis -->
-  <macro name="wheel" params="lr fb tY">
+  <!-- params = left/right XPosition YPosition -->
+  <macro name="wheel" params="lr x_pos y_pos">
     <link name="${lr}_wheel">
       <collision>
-        <origin xyz="0 0 0" rpy="0 ${PI/2} ${PI/2}" />
+        <origin xyz="0 0 0" rpy="${PI/2} 0 0" />
         <geometry>
           <cylinder length="${wheelWidth}" radius="${wheelRadius}"/>
@@ -32,5 +32,5 @@
       </collision>
       <visual>
-        <origin xyz="0 0 0" rpy="0 ${PI/2} ${PI/2}" />
+        <origin xyz="0 0 0" rpy="${PI/2} 0 0 " />
         <geometry>
           <cylinder length="${wheelWidth}" radius="${wheelRadius}"/>
@@ -39,5 +39,5 @@
       </visual>
       <inertial>
-        <origin xyz="0 0 0" rpy="0 ${PI/2} ${PI/2}" />
+        <origin xyz="0 0 0" rpy="${PI/2} 0 0 " />
         <mass value="${wheelMass}"/>
         <cylinder_inertia m="${wheelMass}" r="${wheelRadius}" h="${wheelWidth}"/>
@@ -45,22 +45,25 @@
     </link>
     <gazebo reference="${lr}_wheel">
-      <mu1 value="1.0"/>
-      <mu2 value="1.0"/>
-      <kp  value="10000000.0" />
-      <kd  value="1.0" />
-      <fdir1 value="1 0 0"/>
+      <mu1 value="1"/>
+      <mu2 value="1"/>
+      <kp  value="1000000.0" />
+      <kd  value="10.0" />
+      <fdir1 value="0 0 1"/>
+      <minDepth>0.001</minDepth>
+      <maxContacts>1</maxContacts>
+      <!--maxVel>1.0</maxVel-->
       <material>Gazebo/Red</material>
     </gazebo>
-    <joint name="${lr}_wheel_hinge" type="continuous">
+    <joint name="${lr}_wheel_joint" type="continuous">
       <parent link="chassis"/>
       <child link="${lr}_wheel"/>
-      <origin xyz="${wheelPos*fb} ${tY*wheelWidth/2+tY*chassisWidth/2} ${wheelRadius}" rpy="0 0 0" />
+      <origin xyz="${x_pos} ${y_pos} ${wheelRadius}" rpy="0 0 0" />
       <axis xyz="0 1 0" rpy="0 0 0" />
-      <limit effort="1" velocity="1"/>
-      <joint_properties damping="0.1" friction="0.1"/>
+      <limit effort="100" velocity="100"/>
+      <joint_properties damping="0.0" friction="0.0"/>
     </joint>
     <transmission name="${lr}_trans">
       <type>transmission_interface/SimpleTransmission</type>
-      <joint name="${lr}_wheel_hinge">
+      <joint name="${lr}_wheel_joint">
         <hardwareInterface>EffortJointInterface</hardwareInterface>
       </joint>
